File: pcb/controller/controller.kicad_sch (KiCad schematic)
At the start: 27 parts, among them J1 Conn_01x02, J10 USB_C_Receptacle_USB2.0_16P, J2 Conn_01x02, J3 Conn_01x02, J4 Conn_01x02, J5 Conn_01x02, J6 Conn_01x02, J7 Conn_01x02, J8 RJ45, U2 AP2112K-3.3

Commit message: update controller PCB: wider traces, fix missing trace on V+, add comments, update gerber files
Other:
- note added: "chagelog: 2.2: - wider V+ traces - comments for jumpers - add missing 5V connection when using JST supply"
- title: (none) -> Open Shot Clock Controller
Changed lines of the file:
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@@
 	(generator_version "8.0")
 	(paper "A4")
+	(title_block
+		(title "Open Shot Clock Controller")
+		(rev "2.2")
+	)
 	(junction
 		(at 259.08 147.32)
@@
 		)
 	)
+	(text "chagelog:\n2.2: \n- wider V+ traces\n- comments for jumpers\n- add missing 5V connection when using JST supply"
+		(exclude_from_sim no)
+		(at 187.96 219.202 0)
+		(effects
+			(font
+				(size 1.27 1.27)
+			)
+			(justify left)
+		)
+	)
