File: pcb/display/Display.kicad_sch (KiCad schematic)
At the start: 57 parts, among them J1 XH 2P, J101 RJ45, J102 Screw Terminal 3.5mm, J103 01x08_Pin, J105 U.FL, P101 USB_C_Plug_USB2.0, Q101 2N7002, SW101 SW_4x3mm, SW102 SW_4x3mm, SW103 SW_4x3mm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

Commit message: Changed some Part# for production based on feedback an availability
Parts:
- C2, C3: LCSC Part # C307331 -> C76948
- J103: LCSC Part # (none) -> C6332201
Changed lines of the file:
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@@
 			)
 		)
-		(property "LCSC Part #" "C307331"
+		(property "LCSC Part #" "C76948"
 			(at 20.32 139.7 0)
 			(effects
@@
 			)
 		)
+		(property "LCSC Part #" "C6332201"
+			(at 273.05 124.46 0)
+			(effects
+				(font
+					(size 1.27 1.27)
+				)
+				(hide yes)
+			)
+		)
 		(pin "2"
 		)
@@
 		(at 21.59 190.5 0)
 		(unit 1)
-		(exclude_from_sim yes)
+		(exclude_from_sim no)
 		(in_bom yes)
 		(on_board yes)
@@
 			)
 		)
-		(property "LCSC Part #" "C307331"
+		(property "LCSC Part #" "C76948"
 			(at 30.48 139.7 0)
 			(effects
@@
 		(at 35.56 190.5 0)
 		(unit 1)
-		(exclude_from_sim yes)
+		(exclude_from_sim no)
 		(in_bom yes)
 		(on_board yes)

Commit message: Exclude Symbols from BOM
Parts:
- SYM1, SYM2: now left out of the parts list
Changed lines of the file:
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@@
 		(at 21.59 190.5 0)
 		(unit 1)
-		(exclude_from_sim no)
-		(in_bom yes)
+		(exclude_from_sim yes)
+		(in_bom no)
 		(on_board yes)
 		(dnp no)
@@
 		(at 35.56 190.5 0)
 		(unit 1)
-		(exclude_from_sim no)
-		(in_bom yes)
-		(on_board yes)
-		(dnp no)
+		(exclude_from_sim yes)
+		(in_bom no)
+		(on_board yes)
+		(dnp no)
